Commit message: commit 4-11

File: limo_simulation/model/limo_four_diff.xacro (robot description, xacro)
@@ -1,27 +1,27 @@
 <?xml version="1.0"?>
 <robot name="limo_four_diff" xmlns:xacro="http://ros.org/wiki/xacro">
-    <xacro:arg name="robot_name" default="limo_four_diff"/>
-    <xacro:include filename="$(find limo_simulation)/model/limo_xacro.xacro" />
-    <xacro:include filename="$(find limo_simulation)/model/limo_four_diff.gazebo"/>
-    <!-- Variables -->
-    <xacro:property name="M_PI" value="3.14159"/>
-    <!-- Vehicle Geometries -->
-    <xacro:property name="base_x_size" value="0.13" />
-    <xacro:property name="base_y_size" value="0.12" />
-    <xacro:property name="base_z_size" value="0.1" />
-    <xacro:property name="wheelbase" value="0.2"/>
-    <xacro:property name="track" value="0.13"/>
-    <xacro:property name="wheel_vertical_offset" value="-0.10" />
-    <xacro:property name="base_mass" value="2.1557"/>
-    <xacro:property name="wheel_length" value="0.045" />
-    <xacro:property name="wheel_radius" value="0.045" />
-  <link name="base_footprint"/>
-  <joint name="base_joint" type="fixed">
-    <parent link="base_footprint"/>
-    <child link="base_link"/>
+  <xacro:arg name="robot_name" default="limo_four_diff"/>
+  <xacro:include filename="$(find limo_simulation)/model/limo_xacro.xacro"/>
+  <xacro:include filename="$(find limo_simulation)/model/limo_four_diff.gazebo"/>
+  <!-- Variables -->
+  <xacro:property name="M_PI" value="3.14159"/>
+  <!-- Vehicle Geometries -->
+  <xacro:property name="base_x_size" value="0.13" />
+  <xacro:property name="base_y_size" value="0.12" />
+  <xacro:property name="base_z_size" value="0.1" />
+  <xacro:property name="wheelbase" value="0.2"/>
+  <xacro:property name="track" value="0.13"/>
+  <xacro:property name="wheel_vertical_offset" value="-0.10" />
+  <xacro:property name="base_mass" value="2.1557"/>
+  <xacro:property name="wheel_length" value="0.045" />
+  <xacro:property name="wheel_radius" value="0.045" />
+  <link name="$(arg robot_name)/base_footprint"/>
+  <joint name="$(arg robot_name)/base_joint" type="fixed">
+    <parent link="$(arg robot_name)/base_footprint"/>
+    <child link="$(arg robot_name)/base_link"/>
     <origin xyz="0.0 0.0 0.15" rpy="0 0 0"/>
   </joint>
     <!-- Base link -->
-    <link name="base_link">
+    <link name="$(arg robot_name)/base_link">
         <visual>
             <origin xyz="0 0 -0.15" rpy="0 0 1.57" />
@@ -38,5 +38,5 @@
         </collision>
     </link>
-    <link name="inertial_link">
+    <link name="$(arg robot_name)/inertial_link">
         <inertial>
             <origin xyz="0.0 0.0 0.0" />
@@ -49,26 +49,26 @@
     <joint name="inertial_joint" type="fixed">
         <origin xyz="0 0 0" rpy="0 0 0" />
-        <parent link="base_link" />
-        <child link="inertial_link" />
+        <parent link="$(arg robot_name)/base_link" />
+        <child link="$(arg robot_name)/inertial_link" />
     </joint>
-    <xacro:limo_laser parent_prefix="base_link" frame_prefix="laser">
+    <xacro:limo_laser parent_prefix="$(arg robot_name)/base_link" frame_prefix="$(arg robot_name)/laser">
         <origin xyz="0.103 0 -0.034" rpy="0 0 0"/>
     </xacro:limo_laser>
-    <xacro:limo_depth_camera parent_prefix="base_link" frame_prefix="depth_camera">
+    <xacro:limo_depth_camera parent_prefix="$(arg robot_name)/base_link" frame_prefix="$(arg robot_name)/depth_camera">
         <origin xyz="0.084 0 0.3" rpy="0 0 0"/>
     </xacro:limo_depth_camera>
-    <xacro:limo_imu parent_prefix="base_link" frame_prefix="imu">
+    <xacro:limo_imu parent_prefix="$(arg robot_name)/base_link" frame_prefix="$(arg robot_name)/imu">
         <origin xyz="0.0 0 -0.1" rpy="0 0 0"/>
     </xacro:limo_imu>
-    <xacro:limo_wheel parent_prefix="base_link" wheel_prefix="front_left" reflect="1">
+    <xacro:limo_wheel parent_prefix="$(arg robot_name)/base_link" wheel_prefix="front_left" reflect="1">
         <origin xyz="${wheelbase/2} ${track/2} ${wheel_vertical_offset}" rpy="0 0  0" />
     </xacro:limo_wheel>
-    <xacro:limo_wheel parent_prefix="base_link" wheel_prefix="front_right" reflect="-1">
+    <xacro:limo_wheel parent_prefix="$(arg robot_name)/base_link" wheel_prefix="front_right" reflect="-1">
         <origin xyz="${wheelbase/2} ${-track/2} ${wheel_vertical_offset}" rpy="${M_PI} 0 0" />
     </xacro:limo_wheel>
-    <xacro:limo_wheel parent_prefix="base_link" wheel_prefix="rear_left" reflect="1">
+    <xacro:limo_wheel parent_prefix="$(arg robot_name)/base_link" wheel_prefix="rear_left" reflect="1">
         <origin xyz="${-wheelbase/2} ${track/2} ${wheel_vertical_offset}" rpy="0 0 0" />
     </xacro:limo_wheel>
-    <xacro:limo_wheel parent_prefix="base_link" wheel_prefix="rear_right" reflect="-1">
+    <xacro:limo_wheel parent_prefix="$(arg robot_name)/base_link" wheel_prefix="rear_right" reflect="-1">
         <origin xyz="${-wheelbase/2} ${-track/2} ${wheel_vertical_offset}" rpy="${M_PI} 0 0" />
     </xacro:limo_wheel>
@@ -186,8 +186,8 @@
   </gazebo>
   <gazebo reference="front_left_wheel">
-      <mu1>100</mu1>
-      <mu2>100</mu2>
-      <kp>10000000.0</kp>
-      <kd>1.0</kd>
+      <mu1>1.0</mu1>
+      <mu2>1.0</mu2>
+      <kp>100000.0</kp>
+      <kd>10.0</kd>
       <minDepth>0.01</minDepth>
       <fdir1>1 0 0</fdir1>
@@ -195,8 +195,8 @@
   </gazebo>
   <gazebo reference="front_right_wheel">
-      <mu1>100</mu1>
-      <mu2>100</mu2>
-      <kp>10000000.0</kp>
-      <kd>1.0</kd>
+      <mu1>1.0</mu1>
+      <mu2>1.0</mu2>
+      <kp>100000.0</kp>
+      <kd>10.0</kd>
       <minDepth>0.01</minDepth>
       <fdir1>1 0 0</fdir1>
@@ -204,8 +204,8 @@
   </gazebo>
   <gazebo reference="rear_left_wheel">
-      <mu1>100</mu1>
-      <mu2>100</mu2>
-      <kp>10000000.0</kp>
-      <kd>1.0</kd>
+      <mu1>1.0</mu1>
+      <mu2>1.0</mu2>
+      <kp>100000.0</kp>
+      <kd>10.0</kd>
       <minDepth>0.01</minDepth>
       <fdir1>1 0 0</fdir1>
@@ -213,8 +213,8 @@
   </gazebo>
   <gazebo reference="rear_right_wheel">
-      <mu1>100</mu1>
-      <mu2>100</mu2>
-      <kp>10000000.0</kp>
-      <kd>1.0</kd>
+      <mu1>1.0</mu1>
+      <mu2>1.0</mu2>
+      <kp>100000.0</kp>
+      <kd>10.0</kd>
       <minDepth>0.01</minDepth>
       <fdir1>1 0 0</fdir1>

Commit message: mod for laser_sensor

File: limo_simulation/model/limo_four_diff.xacro (robot description, xacro)
@@ -141,5 +141,5 @@
         </linear_acceleration>
       </imu>
-      <plugin name="$(arg robot_name)_two_wheeled_robot_imu" filename="libgazebo_ros2_imu_sensor.so">
+      <plugin name="$(arg robot_name)_two_wheeled_robot_imu" filename="libgazebo_ros_imu_sensor.so">
         <initial_orientation_as_reference>false</initial_orientation_as_reference>
         <frame_name>imu_link</frame_name>
@@ -151,21 +151,21 @@
     </sensor>
 </gazebo>
-<gazebo reference="laser_link">
-    <sensor name="laser" type="ray">
+<gazebo reference="$(arg robot_name)/laser_link">
+    <sensor name="$(arg robot_name)/laser" type="ray">
       <always_on>true</always_on>
       <visualize>true</visualize>
-      <update_rate>10</update_rate>
+      <update_rate>8</update_rate>
       <ray>
         <scan>
           <horizontal>
-            <samples>120</samples>
+            <samples>720</samples>
             <resolution>1.000000</resolution>
-            <min_angle>-3.14159</min_angle>
-            <max_angle>3.14159</max_angle>
+            <min_angle>-2.09439504</min_angle>
+            <max_angle>2.09439504</max_angle>
           </horizontal>
         </scan>
         <range>
           <min>0.3</min>
-          <max>15.0</max>
+          <max>8.0</max>
           <resolution>0.015</resolution>
         </range>
@@ -176,10 +176,11 @@
         </noise>
       </ray>
-      <plugin name="$(arg robot_name)_scan" filename="libgazebo_ros2_ray_sensor.so">
+      <plugin name="scan" filename="libgazebo_ros_ray_sensor.so">
         <ros>
+          <namespace>$(arg robot_name)</namespace>
           <remapping>~/out:=scan</remapping>
         </ros>
         <output_type>sensor_msgs/LaserScan</output_type>
-        <frame_name>laser_link</frame_name>
+        <frame_name>$(arg robot_name)/laser_link</frame_name>
       </plugin>
     </sensor>

File: limo_simulation/model/limo_xacro.xacro (robot description, xacro)
@@ -45,10 +45,10 @@
                     <cylinder radius="0.02" length="0.01"/>
                 </geometry>
-                <material name='laser_material'>
+                <!--<material name='laser_material'>
                     <ambient>0.1 0.1 0.1 1</ambient>
                     <diffuse>0.1 0.1 0.2 1</diffuse>
                     <specular>0 0 0 0</specular>
                     <emissive>0 0 0 1</emissive>
-                </material>
+                </material>-->
             </visual>
             <collision name='laser_collision'>
@@ -85,10 +85,10 @@
                     <box size="0.02 0.06 0.015"/>
                 </geometry>
-                <material name='depth_camera_material'>
+                <!--<material name='depth_camera_material'>
                     <ambient>0.1 0.1 0.1 1</ambient>
                     <diffuse>0.1 0.1 0.2 1</diffuse>
                     <specular>0 0 0 0</specular>
                     <emissive>0 0 0 1</emissive>
-                </material>
+                </material>-->
             </visual>
             <collision name='depth_camera_collision'>
@@ -131,10 +131,10 @@
                     <box size="0.001 0.001 0.001"/>
                 </geometry>
-                <material name='imu_material'>
+                <!--<material name='imu_material'>
                     <ambient>0.1 0.1 0.1 1</ambient>
                     <diffuse>0.1 0.1 0.2 1</diffuse>
                     <specular>0 0 0 0</specular>
                     <emissive>0 0 0 1</emissive>
-                </material>
+                </material>-->
             </visual>
             <collision name='imu_collision'>
